File: MPU.kicad_sch (KiCad schematic)
At the start: 47 parts, among them J2 Conn_01x02, SW1 SW_DIP_x02, SW3 SW_DIP_x02, SW4 Push, U4 NUC980DKxxYx, Y1 12M, Y2 32.768k

Commit message: update schematic and footprints
Parts:
- removed U4: NUC980DKxxYx, 0_ungrouped:LQFP-128_14x14mm_P0.4mm, symbol 0_ungrouped:NUC980DKxxYx
- added U4: NUC980DKxxYx, Package_QFP:LQFP-128_14x14mm_P0.4mm, symbol SymLibrary:NUC980DKxxYx
- C10, C11, C12, C13, C14, C15, C16, C17, C18, C19, C21, C22, C23, C24, C25, C26, C29, C30, C31, C7, C8, C9: footprint Capacitor_SMD:C_0603_1608Metric -> Capacitor_SMD:C_0805_2012Metric_Pad1.18x1.45mm_HandSolder
- C20, C28, C32, C34: footprint Capacitor_SMD:C_0805_2012Metric -> Capacitor_SMD:C_0805_2012Metric_Pad1.18x1.45mm_HandSolder
- R10, R11, R12, R13, R14, R15, R16, R17, R18, R8, R9: footprint Resistor_SMD:R_0603_1608Metric -> Resistor_SMD:R_0805_2012Metric_Pad1.20x1.40mm_HandSolder
- Y2: footprint 0_ungrouped:Crystal_SMD_3215-2Pin_3.2x1.5mm -> Crystal:Crystal_SMD_3215-2Pin_3.2x1.5mm
Connections:
- net +1V2: now also U4.10 (VDD), U4.118 (VDD), U4.123 (USB0_VDD), U4.13 (VDD), U4.43 (VDD), U4.82 (VDD), U4.94 (VDD)
- net +1V8: now also U4.11 (MVDD), U4.12 (MVDD), U4.83 (MVDD), U4.84 (MVDD)
- net +3V3: now also U4.102 (VDDIO), U4.121 (USB1_VDD33), U4.126 (USB0_VDD33), U4.20 (VDDIO), U4.60 (VDDIO), U4.85 (VDDIO), U4.9 (VDDIO)
- net AVDDADC: now also U4.33 (AVDDADC)
- net GND: now also U4.128 (VSS), U4.32 (AVSSADC), U4.64 (VSS), U4.95 (PLL_VSS)
- net PA0: now also U4.2 (PA.0)
- net PA1: now also U4.3 (PA.1)
- net PA10: now also U4.17 (PA.10)
- net PA11: now also U4.18 (PA.11)
- net PA12: now also U4.19 (PA.12)
- net PA2: now also U4.4 (PA.2)
- net PA3: now also U4.5 (PA.3)
- net PA4: now also U4.6 (PA.4)
- net PA5: now also U4.7 (PA.5)
- net PA6: now also U4.8 (PA.6)
- net PA7: now also U4.14 (PA.7)
- net PA8: now also U4.15 (PA.8)
- net PA9: now also U4.16 (PA.9)
- net PB0: now also U4.29 (PB.0)
- net PB1: now also U4.36 (PB.1)
- net PB13: now also U4.93 (PB.13)
- net PB2: now also U4.38 (PB.2)
- net PB3: now also U4.37 (PB.3)
- net PB4: now also U4.31 (PB.4)
- net PB5: now also U4.35 (PB.5)
- net PB6: now also U4.30 (PB.6)
- net PB7: now also U4.34 (PB.7)
- net PB8: now also U4.42 (PB.8)
- net PC0: now also U4.44 (PC.0)
- net PC1: now also U4.45 (PC.1)
- net PC10: now also U4.54 (PC.10)
- net PC11: now also U4.55 (PC.11)
- net PC12: now also U4.56 (PC.12)
- net PC13: now also U4.57 (PC.13)
- net PC14: now also U4.58 (PC.14)
- net PC15: now also U4.59 (PC.15)
- net PC2: now also U4.46 (PC.2)
- net PC3: now also U4.47 (PC.3)
- net PC4: now also U4.48 (PC.4)
- net PC5: now also U4.49 (PC.5)
- net PC6: now also U4.50 (PC.6)
- net PC7: now also U4.51 (PC.7)
- net PC8: now also U4.52 (PC.8)
- net PC9: now also U4.53 (PC.9)
- net PD10: now also U4.70 (PD.10)
- net PD11: now also U4.71 (PD.11)
- net PD12: now also U4.72 (PD.12)
- net PD13: now also U4.73 (PD.13)
- net PD14: now also U4.74 (PD.14)
- net PD15: now also U4.75 (PD.15)
- net PD2: now also U4.61 (PD.2)
- net PD3: now also U4.62 (PD.3)
- net PD4: now also U4.63 (PD.4)
- net PD5: now also U4.65 (PD.5)
- net PD6: now also U4.66 (PD.6)
- net PD7: now also U4.67 (PD.7)
- net PD8: now also U4.68 (PD.8)
- net PD9: now also U4.69 (PD.9)
- net PE0: now also U4.105 (PE.0)
- net PE1: now also U4.106 (PE.1)
- net PE10: now also U4.115 (PE.10)
- net PE12: now also U4.117 (PE.12)
- net PE2: now also U4.107 (PE.2)
- net PE3: now also U4.108 (PE.3)
- net PE4: now also U4.109 (PE.4)
- net PE5: now also U4.110 (PE.5)
- net PE6: now also U4.111 (PE.6)
- net PE7: now also U4.112 (PE.7)
- net PE8: now also U4.113 (PE.8)
- net PE9: now also U4.114 (PE.9)
- net PF0: now also U4.86 (PF.0)
- net PF1: now also U4.87 (PF.1)
- net PF10: now also U4.99 (PF.10)
- net PF11: now also U4.100 (PF.11)
- net PF12: now also U4.101 (PF.12)
- net PF2: now also U4.88 (PF.2)
- net PF3: now also U4.89 (PF.3)
- net PF4: now also U4.90 (PF.4)
- net PF5: now also U4.91 (PF.5)
- net PF6: now also U4.92 (PF.6)
- net PF7: now also U4.96 (PF.7)
- net PF8: now also U4.97 (PF.8)
- net PF9: now also U4.98 (PF.9)
- net PG0: now also U4.28 (PG.0)
- net PG1: now also U4.27 (PG.1)
- net PG11: now also U4.76 (PG.11)
- net PG12: now also U4.77 (PG.12)
- net PG13: now also U4.78 (PG.13)
- net PG14: now also U4.79 (PG.14)
- net PG15: now also U4.80 (PG.15)
- net PG3: now also U4.26 (PG.3)
- net PG5: now also U4.25 (PG.5)
- net PG6: now also U4.24 (PG.6)
- net PG7: now also U4.23 (PG.7)
- net PG8: now also U4.22 (PG.8)
- net PG9: now also U4.21 (PG.9)
- net USB0_DN: now also U4.124 (USB0_DM)
- net USB0_DP: now also U4.125 (USB0_DP)
- net USB0_REXT: now also U4.127 (USB0_REXT)
- net USB1_DN: now also U4.119 (USB1_DM)
- net USB1_DP: now also U4.120 (USB1_DP)
- net USB1_REXT: now also U4.122 (USB1_REXT)
- net VBAT33: now also U4.39 (VBAT33)
- net VBUS0_VLD: now also U4.116 (PE.11)
- net X32_IN: now also U4.40 (X32_IN)
- net X32_OUT: now also U4.41 (X32_OUT)
- net XT_IN: now also U4.103 (XT_IN)
- net XT_OUT: now also U4.104 (XT_OUT)
- net nRESET: now also U4.81 (nRESET)
- net at R17.1: now also U4.1 (USB0_ID)
